File: pic_programmer/pic_programmer.kicad_sch (KiCad schematic)
At the start: 56 parts, among them J1 DB9-MALE, P1 CONN_2, P101 CONN_1, P102 CONN_1, P103 CONN_1, P104 CONN_1, P105 CONN_1, P106 CONN_1, Q1 BC237, Q2 BC307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

Commit message: Fixed DB9-MALE to DB9-FEMAL
in pic_programmer.kicad_sch
Parts:
- J1: value DB9-MALE -> DB9-FEMAL
Changed lines of the file:
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@@
 			)
 		)
-		(property "Value" "DB9-MALE"
+		(property "Value" "DB9-FEMAL"
 			(at 31.75 77.47 0)
 			(effects
